Commit message: add steer links, edit lidar and camera

File: urdf/camera.xacro (robot description, xacro)
@@ -1,27 +1,40 @@
 <?xml version="1.0"?>
 <robot xmlns:xacro="http://www.ros.org/wiki/xacro">
-    <link name='camera_link'>
-        <visual name='visual'>
-            <origin xyz="0 0 0.0" rpy="0 0 0" />
+    <xacro:property name="camera_x_offset" value="0.75" />
+    <xacro:property name="camera_z_offset" value="0.55" />
+    <link name="camera">
+        <inertial>
+            <mass value="0.1" />
+            <origin rpy="0 0 0" xyz="0 0 0" />
+            <inertia ixx="0.0003866666666666667" ixy="0" ixz="0" iyy="0.00010666666666666668"
+                iyz="0" izz="0.0003866666666666667" />
+        </inertial>
+        <visual>
+            <origin rpy="0 0 0" xyz="0 0 0" />
             <geometry>
-                <box size="0.05 0.1 0.05" />
+                <box size="0.08 0.2 0.08" />
             </geometry>
+            <material name="Blue" />
         </visual>
         <collision>
-            <origin xyz="0 0 0" rpy="0 0 0" />
+            <origin rpy="0 0 0" xyz="0 0 0" />
             <geometry>
-                <box size="0.1 0.1 0.1" />
+                <box size="0.08 0.2 0.08" />
             </geometry>
         </collision>
-        <inertial>
-            <mass value="0.1" />
-            <origin xyz="0 0 0" rpy="0 0 0" />
-            <inertia ixx="0.001" ixy="0.0" ixz="0.0" iyy="0.001" iyz="0.0" izz="0.001" />
-        </inertial>
     </link>
     <joint name="camera_joint" type="fixed">
         <parent link="base_link" />
-        <child link="camera_link" />
-        <origin xyz="1.5 0 0.8" rpy="0 0 0" />
+        <child link="camera" />
+        <origin rpy="0 0 0" xyz="${camera_x_offset} 0 ${camera_z_offset}" />
+    </joint>
+    <!-- Camera Optical Frame -->
+    <link name="camera_optical" />
+    <joint name="camera_optical_joint" type="fixed">
+        <parent link="camera" />
+        <child link="camera_optical" />
+        <!-- Rotate to align with ROS optical frame convention:
+           X: Right, Y: Down, Z: Forward -->
+        <origin rpy="-1.5707963267948966 0 -1.5707963267948966" xyz="0 0 0" />
     </joint>
     <gazebo reference="camera_link">

File: urdf/common_properties.xacro (robot description, xacro)
@@ -1,30 +1,21 @@
 <?xml version="1.0"?>
 <robot xmlns:xacro="http://www.ros.org/wiki/xacro">
-    <xacro:macro name="box_inertia" params="m l w h xyz rpy">
-        <inertial>
-            <origin xyz="${xyz}" rpy="${rpy}"/>
-            <mass value="${m}"/>
-            <inertia ixx="${(m/12) * (h*h + l*l)}" ixy="0" ixz="0"
-                     iyy="${(m/12) * (w*w + l*l)}" iyz="0"
-                     izz="${(m/12) * (w*w + h*h)}"/>
-        </inertial>
-    </xacro:macro>
-    <xacro:macro name="sphere_inertia" params="m r xyz rpy">
-        <inertial>
-            <origin xyz="${xyz}" rpy="${rpy}"/>
-            <mass value="${m}"/>
-            <inertia ixx="${(2*m/5) * (r*r)}" ixy="0" ixz="0"
-                     iyy="${(2*m/5) * (r*r)}" iyz="0"
-                     izz="${(2*m/5) * (r*r)}"/>
-        </inertial>
-    </xacro:macro>
-    <xacro:macro name="cylinder_inertia" params="m r l xyz rpy">
-        <inertial>
-            <origin xyz="${xyz}" rpy="${rpy}"/>
-            <mass value="${m}"/>
-            <inertia ixx="${(m/12) * ((3*r*r) + (l*l))}" ixy="0" ixz="0"
-                     iyy="${(m/12) * ((3*r*r) + (l*l))}" iyz="0"
-                     izz="${(m/2) * (r*r)}"/>
-        </inertial>
-    </xacro:macro>
+  <material name="Gray">
+    <color rgba="0.5 0.5 0.5 1.0"/>
+  </material>
+  <material name="Black">
+    <color rgba="0.0 0.0 0.0 1.0"/>
+  </material>
+  <material name="Red">
+    <color rgba="1.0 0.0 0.0 1.0"/>
+  </material>
+  <material name="Blue">
+    <color rgba="0.0 0.0 1.0 1.0"/>
+  </material>
+  <material name="Green">
+    <color rgba="0.0 1.0 0.0 1.0"/>
+  </material>
+  <material name="White">
+    <color rgba="1.0 1.0 1.0 1.0"/>
+  </material>
 </robot>

File: urdf/ray.xacro (robot description, xacro)
@@ -1,29 +1,32 @@
 <?xml version="1.0"?>
 <robot xmlns:xacro="http://www.ros.org/wiki/xacro">
-    <link name="base_scan">
+    <xacro:property name="laser_radius" value="0.1" />
+    <xacro:property name="laser_length" value="0.08" />
+    <xacro:property name="laser_z_offset" value="0.2" />
+    <link name="lidar">
+        <inertial>
+            <mass value="0.2" />
+            <origin rpy="0 0 0" xyz="0 0 0" />
+            <inertia ixx="0.0006066666666666668" ixy="0" ixz="0" iyy="0.0006066666666666668" iyz="0"
+                izz="0.0010000000000000002" />
+        </inertial>
         <visual>
-            <origin xyz="0 0 0.0" rpy="0 0 0" />
+            <origin rpy="0 0 0" xyz="0 0 0" />
             <geometry>
-                <cylinder length="0.05" radius="0.1" />
+                <cylinder length="${laser_length}" radius="${laser_radius}" />
             </geometry>
+            <material name="Red" />
         </visual>
         <collision>
-            <origin xyz="0 0 0" rpy="0 0 0" />
+            <origin rpy="0 0 0" xyz="0 0 0" />
             <geometry>
-                <cylinder length="0.05" radius="0.1" />
+                <cylinder length="${laser_length}" radius="${laser_radius}" />
             </geometry>
         </collision>
-        <inertial>
-            <mass value="0.114" />
-            <origin xyz="0 0 0" rpy="0 0 0" />
-            <inertia ixx="0.001" ixy="0.0" ixz="0.0"
-                iyy="0.001" iyz="0.0"
-                izz="0.001" />
-        </inertial>
     </link>
-    <joint name="scan_joint" type="fixed">
+    <joint name="lidar_joint" type="fixed">
         <parent link="base_link" />
-        <child link="base_scan" />
-        <origin xyz="1.5 0 0.7" rpy="0 0 0" />
+        <child link="lidar" />
+        <origin rpy="0 0 0" xyz="${base_length/2 + laser_radius} 0 ${laser_z_offset}" />
     </joint>
     <gazebo reference="base_scan">

File: urdf/via.urdf (robot description, URDF)
Before this commit: robot via, 9 links, 8 joints
Links:
- removed link camera
- removed link camera_optical
- removed link lidar
- added link front_left_steer, mass 0.5
- added link front_right_steer, mass 0.5
- link base_link: geometry collision mesh filename=package://via_description/meshes/via_chassis.dae; visual mesh filename=package://via_description/meshes/via_chassis.dae
- link front_left_wheel: geometry collision mesh filename=package://via_description/meshes/tire.dae; visual mesh filename=package://via_description/meshes/tire.dae
- link front_right_wheel: geometry collision mesh filename=package://via_description/meshes/tire.dae; visual mesh filename=package://via_description/meshes/tire.dae
- link rear_left_wheel: geometry collision mesh filename=package://via_description/meshes/tire.dae; visual mesh filename=package://via_description/meshes/tire.dae
- link rear_right_wheel: geometry collision mesh filename=package://via_description/meshes/tire.dae; visual mesh filename=package://via_description/meshes/tire.dae
Joints:
- removed joint camera_joint
- removed joint camera_optical_joint
- removed joint lidar_joint
- added joint front_left_steer_joint: type continuous, parent base_link, child front_left_steer, origin xyz=${front_wheel_x_offset} ${base_width/2 - wheel_length/2} ${-wheel_z_offset} rpy=0 0 0, axis 0 0 1
- added joint front_right_steer_joint: type continuous, parent base_link, child front_right_steer, origin xyz=${front_wheel_x_offset} -${base_width/2 - wheel_length/2} ${-wheel_z_offset} rpy=0 0 0, axis 0 0 1
- joint front_left_joint: origin xyz=1.1483333333333332 0.69 ${-wheel_z_offset} rpy=0 0 0 -> xyz=0 0 0 rpy=0 0 0; parent base_link -> front_left_steer
- joint front_right_joint: origin xyz=1.1483333333333332 -0.69 ${-wheel_z_offset} rpy=0 0 0 -> xyz=0 0 0 rpy=0 0 0; parent base_link -> front_right_steer
- joint rear_left_joint: origin xyz=-1.1483333333333332 0.69 ${-wheel_z_offset} rpy=0 0 0 -> xyz=-${rear_wheel_x_offset} ${base_width/2 - wheel_length/2} ${-wheel_z_offset} rpy=0 0 0
- joint rear_right_joint: origin xyz=-1.1483333333333332 -0.69 ${-wheel_z_offset} rpy=0 0 0 -> xyz=-${rear_wheel_x_offset} -${base_width/2 - wheel_length/2} ${-wheel_z_offset} rpy=0 0 0
