Commit message: 3 saat ugrastiktan sonra aracı artik hareket ettirebiliyoruz

File: urdf/camera.xacro (robot description, xacro)
@@ -38,5 +38,5 @@
         <origin rpy="-1.5707963267948966 0 -1.5707963267948966" xyz="0 0 0" />
     </joint>
-    <gazebo reference="camera_link">
+    <!-- <gazebo reference="camera_link">
         <sensor name='stereo_camera' type='multicamera'>
             <always_on>1</always_on>
@@ -77,4 +77,4 @@
             </plugin>
         </sensor>
-    </gazebo>
+    </gazebo> -->
 </robot>

File: urdf/common_properties.xacro (robot description, xacro)
@@ -1,4 +1,25 @@
 <?xml version="1.0"?>
 <robot xmlns:xacro="http://www.ros.org/wiki/xacro">
+  <xacro:macro name="box_inertia" params="m l w h xyz rpy">
+    <inertial>
+      <origin xyz="${xyz}" rpy="${rpy}"/>
+      <mass value="${m}"/>
+      <inertia ixx="${(m/12) * (h*h + l*l)}" ixy="0" ixz="0" iyy="${(m/12) * (w*w + l*l)}" iyz="0" izz="${(m/12) * (w*w + h*h)}"/>
+    </inertial>
+  </xacro:macro>
+  <xacro:macro name="sphere_inertia" params="m r xyz rpy">
+    <inertial>
+      <origin xyz="${xyz}" rpy="${rpy}"/>
+      <mass value="${m}"/>
+      <inertia ixx="${(2*m/5) * (r*r)}" ixy="0" ixz="0" iyy="${(2*m/5) * (r*r)}" iyz="0" izz="${(2*m/5) * (r*r)}"/>
+    </inertial>
+  </xacro:macro>
+  <xacro:macro name="cylinder_inertia" params="m r l xyz rpy">
+    <inertial>
+      <origin xyz="${xyz}" rpy="${rpy}"/>
+      <mass value="${m}"/>
+      <inertia ixx="${(m/12) * ((3*r*r) + (l*l))}" ixy="0" ixz="0" iyy="${(m/12) * ((3*r*r) + (l*l))}" iyz="0" izz="${(m/2) * (r*r)}"/>
+    </inertial>
+  </xacro:macro>
   <material name="Gray">
     <color rgba="0.5 0.5 0.5 1.0"/>

File: urdf/gps.xacro (robot description, xacro)
@@ -26,12 +26,10 @@
         <axis xyz="0 0 1" />
     </joint>
-    <gazebo reference="gps_link">
+    <!-- <gazebo reference="gps_link">
         <sensor name="gps_sensor" type="gps">
-            <!-- ensure the sensor is active (required) -->
             <always_on>true</always_on>
             <update_rate>100</update_rate>
             <plugin name="gps_plugin" filename="libgazebo_ros_gps_sensor.so">
               <ros>
-                <!-- publish to /gps/data -->
                 <namespace>/gps</namespace>
                 <remapping>~/out:=data</remapping>
@@ -40,4 +38,4 @@
             </plugin>
           </sensor>
-    </gazebo>
+    </gazebo> -->
 </robot>

File: urdf/imu.xacro (robot description, xacro)
@@ -26,12 +26,10 @@
         <axis xyz="0 0 1" />
     </joint>
-    <gazebo reference="imu_link">
+    <!-- <gazebo reference="imu_link">
         <sensor name="imu_sensor" type="imu">
-            <!-- ensure the sensor is active (required) -->
             <always_on>true</always_on>
             <update_rate>100</update_rate>
             <plugin name="imu_plugin" filename="libgazebo_ros_imu_sensor.so">
               <ros>
-                <!-- publish to /imu/data -->
                 <namespace>/imu</namespace>
                 <remapping>~/out:=data</remapping>
@@ -39,4 +37,4 @@
             </plugin>
           </sensor>
-    </gazebo>
+    </gazebo> -->
 </robot>

File: urdf/ray.xacro (robot description, xacro)
@@ -30,5 +30,5 @@
         <origin rpy="0 0 0" xyz="${base_length/2 + laser_radius} 0 ${laser_z_offset}" />
     </joint>
-    <gazebo reference="base_scan">
+    <!-- <gazebo reference="base_scan">
         <material>Gazebo/FlatBlack</material>
         <sensor name="head_hokuyo_sensor_0" type="ray">
@@ -65,4 +65,4 @@
             </plugin>
         </sensor>
-    </gazebo>
+    </gazebo> -->
 </robot>

File: urdf/via.urdf.xacro (robot description, xacro)
@@ -20,11 +20,11 @@
   <xacro:property name="front_wheel_x_offset" value="0.6775" />
   <xacro:property name="rear_wheel_x_offset" value="0.82" />
-  <xacro:property name="wheel_z_offset" value="-0.1" />
+  <xacro:property name="wheel_z_offset" value="0.1" />
   <link name="base_link">
     <inertial>
-      <mass value="500" />
-      <origin rpy="0 0 0" xyz="0 0 0" />
-      <inertia ixx="102.03266666666667" ixy="0" ixz="0" iyy="324.0868333333333" iyz="0"
-        izz="354.3541666666667" />
+      <mass value="1500" />
+      <origin rpy="0 0 0" xyz="0 0 ${base_height/2}" />
+      <inertia ixx="1997.86" ixy="-3e-05" ixz="-1e-06" iyy="442.769" iyz="62.5206"
+        izz="2238.05" />
     </inertial>
     <visual>
@@ -36,5 +36,5 @@
     </visual>
     <collision>
-      <origin rpy="0 0 0" xyz="0 0 ${base_height/2}" />
+      <origin rpy="0 0 1.57" xyz="0 0 ${base_height/2}" />
       <geometry>
         <mesh filename="package://via_description/meshes/via_chassis.dae" />
@@ -42,148 +42,136 @@
     </collision>
   </link>
-  <!-- Fixed Joint between base_footprint and base_link -->
-  <joint name="footprint_to_base" type="fixed">
-    <parent link="base_footprint" />
-    <child link="base_link" />
-    <origin rpy="0 0 0" xyz="0 0 ${wheel_z_offset + base_radius}" />
-  </joint>
-  <link name="front_left_steer">
-    <inertial>
-      <mass value="0.5" />
-      <origin rpy="0 0 0" xyz="0 0 0" />
-      <inertia ixx="0.001" ixy="0" ixz="0" iyy="0.001" iyz="0" izz="0.001" />
-    </inertial>
-  </link>
-  <joint name="front_left_steer_joint" type="continuous">
-    <parent link="base_link" />
-    <child link="front_left_steer" />
-    <origin rpy="0 0 0"
-      xyz="${front_wheel_x_offset} ${base_width/2 - wheel_length/2} ${-wheel_z_offset}" />
-    <axis xyz="0 0 1" />
-  </joint>
-  <link name="front_left_wheel">
-    <inertial>
-      <mass value="0.5" />
-      <origin rpy="1.5707963267948966 0 0" xyz="0 0 0" />
-      <inertia ixx="0.0084125" ixy="0" ixz="0" iyy="0.0084125" iyz="0" izz="0.015625" />
-    </inertial>
-    <visual>
-      <origin rpy="1.5707963267948966 0 3.14" xyz="0 0 0" />
-      <geometry>
-        <mesh filename="package://via_description/meshes/tire.dae" />
-      </geometry>
-      <material name="Black" />
-    </visual>
-    <collision>
-      <origin rpy="1.5707963267948966 0 3.14" xyz="0 0 0" />
-      <geometry>
-        <mesh filename="package://via_description/meshes/tire.dae" />
-      </geometry>
-    </collision>
-  </link>
-  <joint name="front_left_joint" type="continuous">
-    <parent link="front_left_steer" />
-    <child link="front_left_wheel" />
-    <origin rpy="0 0 0" xyz="0 0 0" />
-    <axis xyz="0 1 0" />
-  </joint>
-  <link name="front_right_steer">
-    <inertial>
-      <mass value="0.5" />
-      <origin rpy="0 0 0" xyz="0 0 0" />
-      <inertia ixx="0.001" ixy="0" ixz="0" iyy="0.001" iyz="0" izz="0.001" />
-    </inertial>
-  </link>
-  <joint name="front_right_steer_joint" type="continuous">
-    <parent link="base_link" />
-    <child link="front_right_steer" />
-    <origin rpy="0 0 0"
-      xyz="${front_wheel_x_offset} -${base_width/2 - wheel_length/2} ${-wheel_z_offset}" />
-    <axis xyz="0 0 1" />
-  </joint>
-  <link name="front_right_wheel">
-    <inertial>
-      <mass value="0.5" />
-      <origin rpy="1.5707963267948966 0 0" xyz="0 0 0" />
-      <inertia ixx="0.0084125" ixy="0" ixz="0" iyy="0.0084125" iyz="0" izz="0.015625" />
-    </inertial>
-    <visual>
-      <origin rpy="1.5707963267948966 0 3.14" xyz="0 0 0" />
-      <geometry>
-        <mesh filename="package://via_description/meshes/tire.dae" />
-      </geometry>
-      <material name="Black" />
-    </visual>
-    <collision>
-      <origin rpy="1.5707963267948966 0 3.14" xyz="0 0 0" />
-      <geometry>
-        <mesh filename="package://via_description/meshes/tire.dae" />
-      </geometry>
-    </collision>
-  </link>
-  <joint name="front_right_joint" type="continuous">
-    <parent link="front_right_steer" />
-    <child link="front_right_wheel" />
-    <origin rpy="0 0 0" xyz="0 0 0" />
-    <axis xyz="0 1 0" />
-  </joint>
-  <link name="rear_left_wheel">
-    <inertial>
-      <mass value="0.5" />
-      <origin rpy="1.5707963267948966 0 0" xyz="0 0 0" />
-      <inertia ixx="0.0084125" ixy="0" ixz="0" iyy="0.0084125" iyz="0" izz="0.015625" />
-    </inertial>
-    <visual>
-      <origin rpy="1.5707963267948966 0 0" xyz="0 0 0" />
-      <geometry>
-        <mesh filename="package://via_description/meshes/tire.dae" />
-      </geometry>
-      <material name="Black" />
-    </visual>
-    <collision>
-      <origin rpy="1.5707963267948966 0 0" xyz="0 0 0" />
-      <geometry>
-        <mesh filename="package://via_description/meshes/tire.dae" />
-      </geometry>
-    </collision>
-  </link>
-  <joint name="rear_left_joint" type="continuous">
-    <parent link="base_link" />
-    <child link="rear_left_wheel" />
-    <origin rpy="0 0 0"
-      xyz="-${rear_wheel_x_offset} ${base_width/2 - wheel_length/2} ${-wheel_z_offset}" />
-    <axis xyz="0 1 0" />
-  </joint>
-  <link name="rear_right_wheel">
-    <inertial>
-      <mass value="0.5" />
-      <origin rpy="1.5707963267948966 0 0" xyz="0 0 0" />
-      <inertia ixx="0.0084125" ixy="0" ixz="0" iyy="0.0084125" iyz="0" izz="0.015625" />
-    </inertial>
-    <visual>
-      <origin rpy="1.5707963267948966 0 0" xyz="0 0 0" />
-      <geometry>
-        <mesh filename="package://via_description/meshes/tire.dae" />
-      </geometry>
-      <material name="Black" />
-    </visual>
-    <collision>
-      <origin rpy="1.5707963267948966 0 0" xyz="0 0 0" />
-      <geometry>
-        <mesh filename="package://via_description/meshes/tire.dae" />
-      </geometry>
-    </collision>
-  </link>
-  <joint name="rear_right_joint" type="continuous">
-    <parent link="base_link" />
-    <child link="rear_right_wheel" />
-    <origin rpy="0 0 0"
-      xyz="-${rear_wheel_x_offset} -${base_width/2 - wheel_length/2} ${-wheel_z_offset}" />
-    <axis xyz="0 1 0" />
-  </joint>
-  <xacro:include filename="ray.xacro" />
+    <link name="rear_right_axle">
+        <visual>
+            <geometry>
+                <mesh filename="package://via_description/meshes/tire.dae" />
+            </geometry>
+            <origin xyz="0 0 0" rpy="${pi / 2.0} 0 0" />
+        </visual>
+        <xacro:cylinder_inertia m="30" r="${base_radius*2}" l="${wheel_length}"
+            xyz="0 0 0" rpy="${pi / 2.0} 0 0" />
+        <collision>
+            <geometry>
+                <cylinder radius="${base_radius}" length="${wheel_length}" />
+            </geometry>
+            <origin xyz="0 0 0" rpy="${pi / 2.0} 0 0" />
+        </collision>
+    </link>
+    <link name="rear_left_axle">
+        <visual>
+            <geometry>
+                <mesh filename="package://via_description/meshes/tire.dae" />
+            </geometry>
+            <origin xyz="0 0 0" rpy="${pi / 2.0} 0 0" />
+        </visual>
+        <xacro:cylinder_inertia m="30" r="${base_radius*2}" l="${wheel_length}"
+            xyz="0 0 0" rpy="${pi / 2.0} 0 0" />
+        <collision>
+            <geometry>
+                <cylinder radius="${base_radius}" length="${wheel_length}" />
+            </geometry>
+            <origin xyz="0 0 0" rpy="${pi / 2.0} 0 0" />
+        </collision>
+    </link>
+    <link name="front_right_steer">
+        <inertial>
+            <origin rpy="0 0 0" xyz="0.003381 1.5929e-07 0.02162" />
+            <mass value="1" />
+            <inertia ixx="1.0" ixy="0.0" ixz="0.0" iyy="1.0" iyz="0.0" izz="1.0" />
+        </inertial>
+    </link>
+    <link name="front_right_axle">
+        <visual>
+            <geometry>
+                <mesh filename="package://via_description/meshes/tire.dae" />
+            </geometry>
+            <origin xyz="0 0 0" rpy="${pi / 2.0} 0 0" />
+        </visual>
+        <xacro:cylinder_inertia m="30" r="${base_radius*2}" l="${wheel_length}"
+            xyz="0 0 0" rpy="${pi / 2.0} 0 0" />
+        <collision>
+            <geometry>
+                <cylinder radius="${base_radius}" length="${wheel_length}" />
+            </geometry>
+            <origin xyz="0 0 0" rpy="${pi / 2.0} 0 0" />
+        </collision>
+    </link>
+    <link name="front_left_steer">
+        <inertial>
+            <origin rpy="0 0 0" xyz="0.003381 1.5929e-07 0.02162" />
+            <mass value="1" />
+            <inertia ixx="1.0" ixy="0.0" ixz="0.0" iyy="1.0" iyz="0.0" izz="1.0" />
+        </inertial>
+    </link>
+    <link name="front_left_axle">
+        <visual>
+            <geometry>
+                <mesh filename="package://via_description/meshes/tire.dae" />
+            </geometry>
+            <origin xyz="0 0 0" rpy="${pi / 2.0} 0 0" />
+        </visual>
+        <xacro:cylinder_inertia m="30" r="${base_radius*2}" l="${wheel_length}"
+            xyz="0 0 0" rpy="${pi / 2.0} 0 0" />
+        <collision>
+            <geometry>
+                <cylinder radius="${base_radius}" length="${wheel_length}" />
+            </geometry>
+            <origin xyz="0 0 0" rpy="${pi / 2.0} 0 0" />
+        </collision>
+    </link>
+    <joint name="base_joint" type="fixed">
+        <parent link="base_footprint" />
+        <child link="base_link" />
+        <origin xyz="0 0 ${base_radius-wheel_z_offset}" rpy="0 0 0" />
+    </joint>
+    <joint name="rear_right_axle_joint" type="continuous">
+        <parent link="base_link" />
+        <child link="rear_right_axle" />
+        <origin
+            xyz="${-rear_wheel_x_offset} ${-(base_width / 2.0) + (wheel_length / 2.0)} ${wheel_z_offset}"
+            rpy="0 0 0" />
+        <axis xyz="0 1 0" />
+    </joint>
+    <joint name="rear_left_axle_joint" type="continuous">
+        <parent link="base_link" />
+        <child link="rear_left_axle" />
+        <origin
+            xyz="${-rear_wheel_x_offset} ${(base_width / 2.0) - (wheel_length / 2.0)} ${wheel_z_offset}"
+            rpy="0 0 0" />
+        <axis xyz="0 1 0" />
+    </joint>
+    <joint name="front_right_steer_joint" type="continuous">
+        <parent link="base_link" />
+        <child link="front_right_steer" />
+        <origin
+            xyz="${front_wheel_x_offset} ${-(base_width / 2.0) + (wheel_length / 2.0)} ${wheel_z_offset}"
+            rpy="0 0 0" />
+        <axis xyz="0 0 1" />
+    </joint>
+    <joint name="front_right_axle_joint" type="continuous">
+        <parent link="front_right_steer" />
+        <child link="front_right_axle" />
+        <origin xyz="0 0 0" rpy="0 0 0" />
+        <axis xyz="0 1 0" />
+    </joint>
+    <joint name="front_left_steer_joint" type="continuous">
+        <parent link="base_link" />
+        <child link="front_left_steer" />
+        <origin
+            xyz="${front_wheel_x_offset} ${(base_width / 2.0) - (wheel_length / 2.0)} ${wheel_z_offset}"
+            rpy="0 0 0" />
+        <axis xyz="0 0 1" />
+    </joint>
+    <joint name="front_left_axle_joint" type="continuous">
+        <parent link="front_left_steer" />
+        <child link="front_left_axle" />
+        <origin xyz="0 0 0" rpy="0 0 0" />
+        <axis xyz="0 1 0" />
+    </joint>
+  <!-- <xacro:include filename="ray.xacro" />
   <xacro:include filename="camera.xacro" />
   <xacro:include filename="imu.xacro" />
   <xacro:include filename="gps.xacro" />
-  <xacro:include filename="distance.xacro" />
+  <xacro:include filename="distance.xacro" /> -->
+  <xacro:include filename="via_gazebo.xacro" />
 </robot>

File: urdf/via_gazebo.xacro (robot description, xacro)
@@ -19,5 +19,5 @@
             <max_speed>20</max_speed>
             <!-- PID tuning -->
-            <left_steering_pid_gain>2000 0 100</left_steering_pid_gain>
+            <left_steering_pid_gain>1500 0 150</left_steering_pid_gain>
             <left_steering_i_range>0 0</left_steering_i_range>
             <right_steering_pid_gain>2000 0 100</right_steering_pid_gain>

Commit message: add gps, imu, camera and scan sensors

File: urdf/camera.xacro (robot description, xacro)
@@ -3,10 +3,9 @@
     <xacro:property name="camera_x_offset" value="0.75" />
     <xacro:property name="camera_z_offset" value="0.55" />
-    <link name="camera">
+    <link name="camera_link">
         <inertial>
             <mass value="0.1" />
             <origin rpy="0 0 0" xyz="0 0 0" />
-            <inertia ixx="0.0003866666666666667" ixy="0" ixz="0" iyy="0.00010666666666666668"
-                iyz="0" izz="0.0003866666666666667" />
+            <inertia ixx="0.0003866666666666667" ixy="0" ixz="0" iyy="0.00010666666666666668" iyz="0" izz="0.0003866666666666667" />
         </inertial>
         <visual>
@@ -26,5 +25,5 @@
     <joint name="camera_joint" type="fixed">
         <parent link="base_link" />
-        <child link="camera" />
+        <child link="camera_link" />
         <origin rpy="0 0 0" xyz="${camera_x_offset} 0 ${camera_z_offset}" />
     </joint>
@@ -32,5 +31,5 @@
     <link name="camera_optical" />
     <joint name="camera_optical_joint" type="fixed">
-        <parent link="camera" />
+        <parent link="camera_link" />
         <child link="camera_optical" />
         <!-- Rotate to align with ROS optical frame convention:
@@ -38,24 +37,10 @@
         <origin rpy="-1.5707963267948966 0 -1.5707963267948966" xyz="0 0 0" />
     </joint>
-    <!-- <gazebo reference="camera_link">
-        <sensor name='stereo_camera' type='multicamera'>
+    <gazebo reference="camera_link">
+        <sensor name='camera_sensor' type='camera'>
             <always_on>1</always_on>
             <update_rate>100</update_rate>
-            <camera name='left'>
-                <pose>0 -0.12 0 0 -0 0</pose>
-                <horizontal_fov>1.91986</horizontal_fov>
-                <image>
-                    <width>672</width>
-                    <height>376</height>
-                    <format>R8G8B8</format>
-                </image>
-                <clip>
-                    <near>0.3</near>
-                    <far>130</far>
-                </clip>
-                <vertical_fov>1.2217304764</vertical_fov>
-            </camera>
-            <camera name='right'>
-                <pose>0 0.12 0 0 -0 0</pose>
+            <camera name='camera0'>
+                <pose>0 0 0 0 -0 0</pose>
                 <horizontal_fov>1.91986</horizontal_fov>
                 <image>
@@ -77,4 +62,4 @@
             </plugin>
         </sensor>
-    </gazebo> -->
+    </gazebo>
 </robot>

File: urdf/gps.xacro (robot description, xacro)
@@ -26,5 +26,5 @@
         <axis xyz="0 0 1" />
     </joint>
-    <!-- <gazebo reference="gps_link">
+    <gazebo reference="gps_link">
         <sensor name="gps_sensor" type="gps">
             <always_on>true</always_on>
@@ -38,4 +38,4 @@
             </plugin>
           </sensor>
-    </gazebo> -->
+    </gazebo>
 </robot>

File: urdf/imu.xacro (robot description, xacro)
@@ -26,5 +26,5 @@
         <axis xyz="0 0 1" />
     </joint>
-    <!-- <gazebo reference="imu_link">
+    <gazebo reference="imu_link">
         <sensor name="imu_sensor" type="imu">
             <always_on>true</always_on>
@@ -37,4 +37,4 @@
             </plugin>
           </sensor>
-    </gazebo> -->
+    </gazebo>
 </robot>

File: urdf/ray.xacro (robot description, xacro)
@@ -4,5 +4,5 @@
     <xacro:property name="laser_length" value="0.08" />
     <xacro:property name="laser_z_offset" value="0.2" />
-    <link name="lidar">
+    <link name="base_scan">
         <inertial>
             <mass value="0.2" />
@@ -27,8 +27,8 @@
     <joint name="lidar_joint" type="fixed">
         <parent link="base_link" />
-        <child link="lidar" />
+        <child link="base_scan" />
         <origin rpy="0 0 0" xyz="${base_length/2 + laser_radius} 0 ${laser_z_offset}" />
     </joint>
-    <!-- <gazebo reference="base_scan">
+    <gazebo reference="base_scan">
         <material>Gazebo/FlatBlack</material>
         <sensor name="head_hokuyo_sensor_0" type="ray">
@@ -47,5 +47,5 @@
                 <range>
                     <min>0.120000</min>
-                    <max>30.0</max>
+                    <max>12.0</max>
                     <resolution>0.010</resolution>
                 </range>
@@ -65,4 +65,4 @@
             </plugin>
         </sensor>
-    </gazebo> -->
+    </gazebo>
 </robot>

File: urdf/via.urdf.xacro (robot description, xacro)
@@ -169,9 +169,9 @@
         <axis xyz="0 1 0" />
     </joint>
-  <!-- <xacro:include filename="ray.xacro" />
+  <xacro:include filename="ray.xacro" />
   <xacro:include filename="camera.xacro" />
   <xacro:include filename="imu.xacro" />
   <xacro:include filename="gps.xacro" />
-  <xacro:include filename="distance.xacro" /> -->
+  <xacro:include filename="distance.xacro" />
   <xacro:include filename="via_gazebo.xacro" />
 </robot>

Commit message: add depth camera and fix camera position

File: urdf/camera.xacro (robot description, xacro)
@@ -1,6 +1,6 @@
 <?xml version="1.0"?>
 <robot xmlns:xacro="http://www.ros.org/wiki/xacro">
-    <xacro:property name="camera_x_offset" value="0.75" />
-    <xacro:property name="camera_z_offset" value="0.55" />
+    <xacro:property name="camera_x_offset" value="1.25" />
+    <xacro:property name="camera_z_offset" value="0.50" />
     <link name="camera_link">
         <inertial>
@@ -59,5 +59,5 @@
                     <namespace>zed_cam</namespace>
                 </ros>
-                <frame_name>camera_link</frame_name>
+                <frame_name>camera_optical</frame_name>
             </plugin>
         </sensor>

File: urdf/depth.xacro (robot description, xacro)
@@ -23,5 +23,5 @@
                     <namespace>zed_cam</namespace>
                 </ros>
-                <frame_name>camera_link</frame_name>
+                <frame_name>camera_optical</frame_name>
             </plugin>
         </sensor>

File: urdf/via.urdf.xacro (robot description, xacro)
@@ -165,4 +165,5 @@
   <xacro:include filename="gps.xacro" />
   <xacro:include filename="distance.xacro" />
+  <xacro:include filename="depth.xacro" />
   <xacro:include filename="via_gazebo.xacro" />
 </robot>

Commit message: change camera location

File: urdf/camera.xacro (robot description, xacro)
@@ -1,6 +1,6 @@
 <?xml version="1.0"?>
 <robot xmlns:xacro="http://www.ros.org/wiki/xacro">
-    <xacro:property name="camera_x_offset" value="1.25" />
-    <xacro:property name="camera_z_offset" value="0.50" />
+    <xacro:property name="camera_x_offset" value="0.25" />
+    <xacro:property name="camera_z_offset" value="0.85" />
     <link name="camera_link">
         <inertial>
