Commit message: change lidar range

File: urdf/ray.xacro (robot description, xacro)
@@ -1,5 +1,5 @@
 <?xml version="1.0"?>
 <robot xmlns:xacro="http://www.ros.org/wiki/xacro">
-    <xacro:property name="laser_radius" value="0.1" />
+    <xacro:property name="laser_radius" value="0.055" />
     <xacro:property name="laser_length" value="0.08" />
     <xacro:property name="laser_z_offset" value="0.2" />
@@ -18,10 +18,4 @@
             <material name="Red" />
         </visual>
-        <collision>
-            <origin rpy="0 0 0" xyz="0 0 0" />
-            <geometry>
-                <cylinder length="${laser_length}" radius="${laser_radius}" />
-            </geometry>
-        </collision>
     </link>
     <joint name="lidar_joint" type="fixed">
