Commit message: fix robot sliding

File: urdf/via.urdf.xacro (robot description, xacro)
@@ -1,36 +1,33 @@
 <?xml version="1.0"?>
 <robot name="via"
-  xmlns:xacro="http://www.ros.org/wiki/xacro">
-  <link name="base_footprint" />
-  <xacro:include filename="common_properties.xacro" />
-  <xacro:property name="base_length" value="2.63" />
-  <xacro:property name="base_width" value="1.26" />
-  <xacro:property name="base_height" value="0.928" />
-  <xacro:property name="base_radius" value="0.25" />
-  <xacro:property name="wheel_length" value="0.12" />
-  <xacro:property name="front_wheel_x_offset" value="0.6775" />
-  <xacro:property name="rear_wheel_x_offset" value="0.82" />
-  <xacro:property name="wheel_z_offset" value="0.1" />
-  <link name="base_link">
-    <inertial>
-      <mass value="1500" />
-      <origin rpy="0 0 0" xyz="0 0 ${base_height/2}" />
-      <inertia ixx="1997.86" ixy="-3e-05" ixz="-1e-06" iyy="442.769" iyz="62.5206"
-        izz="2238.05" />
-    </inertial>
-    <visual>
-      <origin rpy="0 0 1.57" xyz="0 0 ${base_height/2}" />
-      <geometry>
-        <mesh filename="package://via_description/meshes/via_chassis.dae" />
-      </geometry>
-      <material name="Gray" />
-    </visual>
-    <collision>
-      <origin rpy="0 0 1.57" xyz="0 0 ${base_height/2}" />
-      <geometry>
-        <mesh filename="package://via_description/meshes/via_chassis.dae" />
-      </geometry>
-    </collision>
-  </link>
+    xmlns:xacro="http://www.ros.org/wiki/xacro">
+    <link name="base_footprint" />
+    <xacro:include filename="inertial_macros.xacro" />
+    <xacro:property name="base_length" value="2.63" />
+    <xacro:property name="base_width" value="1.26" />
+    <xacro:property name="base_height" value="0.928" />
+    <xacro:property name="base_radius" value="0.25" />
+    <xacro:property name="wheel_length" value="0.12" />
+    <xacro:property name="front_wheel_x_offset" value="0.6775" />
+    <xacro:property name="rear_wheel_x_offset" value="0.82" />
+    <xacro:property name="wheel_z_offset" value="0.1" />
+    <link name="base_link">
+        <xacro:inertial_box mass="100" x="${base_length}" y="${base_width}" z="${base_height}">
+            <origin xyz="0 0 ${base_height/2}" rpy="0 0 0" />
+        </xacro:inertial_box>
+        <visual>
+            <origin rpy="0 0 1.57" xyz="0 0 ${base_height/2}" />
+            <geometry>
+                <mesh filename="package://via_description/meshes/via_chassis.dae" />
+            </geometry>
+            <material name="Gray" />
+        </visual>
+        <collision>
+            <origin rpy="0 0 1.57" xyz="0 0 ${base_height/2}" />
+            <geometry>
+                <mesh filename="package://via_description/meshes/via_chassis.dae" />
+            </geometry>
+        </collision>
+    </link>
     <link name="rear_right_axle">
         <visual>
@@ -40,6 +37,9 @@
             <origin xyz="0 0 0" rpy="${pi / 2.0} 0 0" />
         </visual>
-        <xacro:cylinder_inertia m="30" r="${base_radius*2}" l="${wheel_length}"
-            xyz="0 0 0" rpy="${pi / 2.0} 0 0" />
+        <!-- <xacro:cylinder_inertia m="30" r="${base_radius*2}" l="${wheel_length}"
+            xyz="0 0 0" rpy="${pi / 2.0} 0 0" /> -->
+        <xacro:inertial_cylinder mass="10" length="${wheel_length}" radius="${base_radius}">
+            <origin xyz="0 0 0" rpy="${pi / 2.0} 0 0" />
+        </xacro:inertial_cylinder>
         <collision>
             <geometry>
@@ -56,6 +56,9 @@
             <origin xyz="0 0 0" rpy="${pi / 2.0} 0 0" />
         </visual>
-        <xacro:cylinder_inertia m="30" r="${base_radius*2}" l="${wheel_length}"
-            xyz="0 0 0" rpy="${pi / 2.0} 0 0" />
+        <!-- <xacro:cylinder_inertia m="30" r="${base_radius*2}" l="${wheel_length}"
+            xyz="0 0 0" rpy="${pi / 2.0} 0 0" /> -->
+        <xacro:inertial_cylinder mass="10" length="${wheel_length}" radius="${base_radius}">
+            <origin xyz="0 0 0" rpy="${pi / 2.0} 0 0" />
+        </xacro:inertial_cylinder>
         <collision>
             <geometry>
@@ -69,5 +72,5 @@
             <origin rpy="0 0 0" xyz="0.003381 1.5929e-07 0.02162" />
             <mass value="1" />
-            <inertia ixx="1.0" ixy="0.0" ixz="0.0" iyy="1.0" iyz="0.0" izz="1.0" />
+            <inertia ixx="0.01" ixy="0.0" ixz="0.0" iyy="0.01" iyz="0.0" izz="0.01" />
         </inertial>
     </link>
@@ -79,6 +82,9 @@
             <origin xyz="0 0 0" rpy="${pi / 2.0} 0 0" />
         </visual>
-        <xacro:cylinder_inertia m="30" r="${base_radius*2}" l="${wheel_length}"
-            xyz="0 0 0" rpy="${pi / 2.0} 0 0" />
+        <!-- <xacro:cylinder_inertia m="30" r="${base_radius*2}" l="${wheel_length}"
+            xyz="0 0 0" rpy="${pi / 2.0} 0 0" /> -->
+        <xacro:inertial_cylinder mass="10" length="${wheel_length}" radius="${base_radius}">
+            <origin xyz="0 0 0" rpy="${pi / 2.0} 0 0" />
+        </xacro:inertial_cylinder>
         <collision>
             <geometry>
@@ -92,5 +98,5 @@
             <origin rpy="0 0 0" xyz="0.003381 1.5929e-07 0.02162" />
             <mass value="1" />
-            <inertia ixx="1.0" ixy="0.0" ixz="0.0" iyy="1.0" iyz="0.0" izz="1.0" />
+            <inertia ixx="0.01" ixy="0.0" ixz="0.0" iyy="0.01" iyz="0.0" izz="0.01" />
         </inertial>
     </link>
@@ -102,6 +108,9 @@
             <origin xyz="0 0 0" rpy="${pi / 2.0} 0 0" />
         </visual>
-        <xacro:cylinder_inertia m="30" r="${base_radius*2}" l="${wheel_length}"
-            xyz="0 0 0" rpy="${pi / 2.0} 0 0" />
+        <!-- <xacro:cylinder_inertia m="30" r="${base_radius*2}" l="${wheel_length}"
+            xyz="0 0 0" rpy="${pi / 2.0} 0 0" /> -->
+        <xacro:inertial_cylinder mass="10" length="${wheel_length}" radius="${base_radius}">
+            <origin xyz="0 0 0" rpy="${pi / 2.0} 0 0" />
+        </xacro:inertial_cylinder>
         <collision>
             <geometry>
@@ -160,10 +169,10 @@
         <axis xyz="0 1 0" />
     </joint>
-  <xacro:include filename="ray.xacro" />
-  <xacro:include filename="camera.xacro" />
-  <xacro:include filename="imu.xacro" />
-  <xacro:include filename="gps.xacro" />
-  <xacro:include filename="distance.xacro" />
-  <xacro:include filename="depth.xacro" />
-  <xacro:include filename="via_gazebo.xacro" />
+    <xacro:include filename="ray.xacro" />
+    <xacro:include filename="camera.xacro" />
+    <xacro:include filename="imu.xacro" />
+    <xacro:include filename="gps.xacro" />
+    <xacro:include filename="distance.xacro" />
+    <xacro:include filename="depth.xacro" />
+    <xacro:include filename="via_gazebo.xacro" />
 </robot>

File: urdf/via_gazebo.xacro (robot description, xacro)
@@ -19,9 +19,9 @@
             <max_speed>20</max_speed>
             <!-- PID tuning -->
-            <left_steering_pid_gain>1500 0 150</left_steering_pid_gain>
+            <left_steering_pid_gain>100 0 150</left_steering_pid_gain>
             <left_steering_i_range>0 0</left_steering_i_range>
-            <right_steering_pid_gain>2000 0 100</right_steering_pid_gain>
+            <right_steering_pid_gain>100 0 100</right_steering_pid_gain>
             <right_steering_i_range>0 0</right_steering_i_range>
-            <linear_velocity_pid_gain>1000 0 1</linear_velocity_pid_gain>
+            <linear_velocity_pid_gain>500 0 1</linear_velocity_pid_gain>
             <linear_velocity_i_range>0 0</linear_velocity_i_range>
             <!-- output -->

Commit message: araç tekerleri döndürüldü araç hareketi düzeltildi

File: urdf/via.urdf.xacro (robot description, xacro)
@@ -54,5 +54,5 @@
                 <mesh filename="package://via_description/meshes/tire.dae" />
             </geometry>
-            <origin xyz="0 0 0" rpy="${pi / 2.0} 0 0" />
+            <origin xyz="0 0 0" rpy="${pi / 2.0} 0 ${pi}" />
         </visual>
         <!-- <xacro:cylinder_inertia m="30" r="${base_radius*2}" l="${wheel_length}"
@@ -106,5 +106,5 @@
                 <mesh filename="package://via_description/meshes/tire.dae" />
             </geometry>
-            <origin xyz="0 0 0" rpy="${pi / 2.0} 0 0" />
+            <origin xyz="0 0 0" rpy="${pi / 2.0} 0 ${pi}" />
         </visual>
         <!-- <xacro:cylinder_inertia m="30" r="${base_radius*2}" l="${wheel_length}"
@@ -130,5 +130,5 @@
         <origin
             xyz="${-rear_wheel_x_offset} ${-(base_width / 2.0) + (wheel_length / 2.0)} ${wheel_z_offset}"
-            rpy="0 0 3.1416" />
+            rpy="0 0 0" />
         <axis xyz="0 1 0" />
     </joint>
@@ -146,5 +146,5 @@
         <origin
             xyz="${front_wheel_x_offset} ${-(base_width / 2.0) + (wheel_length / 2.0)} ${wheel_z_offset}"
-            rpy="0 0 3.1416" />
+            rpy="0 0 0" />
         <axis xyz="0 0 1" />
     </joint>
